Commit message: 20260908新增自主探索建图和双激光雷达融合

File: install/diff_drive_gazebo/share/diff_drive_gazebo/urdf/robot2.urdf (robot description, URDF)
Before this commit: robot diff_drive, 7 links, 6 joints
Links:
- removed link laser
- added link laser_back, mass 0.1; collision cylinder length=0.05 radius=0.03; visual cylinder length=0.05 radius=0.03
- added link laser_front, mass 0.1; collision cylinder length=0.05 radius=0.03; visual cylinder length=0.05 radius=0.03
Joints:
- removed joint laser_joint
- added joint laser_back_joint: type fixed, parent base_link, child laser_back, origin xyz=-0.15 0 0.1 rpy=0 0 3.14159
- added joint laser_front_joint: type fixed, parent base_link, child laser_front, origin xyz=0.15 0 0.1 rpy=0 0 0
